File: shield-pcb/chibi-cw.kicad_pcb (KiCad board)
At the start: 2 copper layers, 48.3 x 53.3 mm, 59 parts, among them J1 HEADPHONES, K1 CONN_3, K2 CONN_3, P1 CONN_4, P2 CONN_4, P3 CONN_2, P4 SPEAKER, Q1 BC847, U1 TPA6130A2

Commit message: Trivial changes, here and there.
Parts:
- moved R20 0.50 mm to (48.5, 52.5)
Routing:
- net N-0000024: track 18.9 -> 19.4 mm
- net IO9: track 26.5 -> 26.0 mm
Changed lines of the file:
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@@
   )
   (module SM0603 (layer F.Cu)
-    (at 48.5 53 270)
+    (at 48.5 52.5 270)
     (attr smd)
     (fp_text reference R20 (at 2 0 360) (layer F.SilkS)
@@
   (segment (start 46.736 29.514) (end 46.736 27.94) (width 0.254) (layer F.Cu) (net 13))
   (segment (start 45.75 30.5) (end 46.736 29.514) (width 0.254) (layer F.Cu) (net 13))
-  (segment (start 48.5 52.238) (end 48.5 47.5) (width 0.254) (layer F.Cu) (net 14))
+  (segment (start 48.5 51.738) (end 48.5 47.5) (width 0.254) (layer F.Cu) (net 14) (status 10))
   (segment (start 44.196 30.446) (end 44.196 27.94) (width 0.254) (layer B.Cu) (net 14))
   (via (at 48.5 47.5) (size 0.889) (layers F.Cu B.Cu) (net 14))
@@
   (segment (start 54.2 57.4) (end 54.8 58) (width 0.254) (layer F.Cu) (net 26))
   (segment (start 62.00038 59.99898) (end 55.50102 59.99898) (width 0.254) (layer F.Cu) (net 27))
-  (segment (start 48.5 58.5) (end 48.5 53.762) (width 0.254) (layer F.Cu) (net 27))
+  (segment (start 48.5 58.5) (end 48.5 53.262) (width 0.254) (layer F.Cu) (net 27) (status 20))
   (via (at 48.5 58.5) (size 0.889) (layers F.Cu B.Cu) (net 27))
   (segment (start 50 60) (end 48.5 58.5) (width 0.254) (layer B.Cu) (net 27))
